File: 20kN_dev.kicad_sch (KiCad schematic)
At the start: 18 parts, among them IC1 STM32L476RGT6, IC2 DRV8834PWPR, J1 Conn_ARM_JTAG_SWD_10, J2 USB_C_Receptacle_PowerOnly_6P, J3 1757242, J4 RJ45_Abracon_ARJP11A-MASA-B-A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, J5 690367180672, J6 RJ45_Abracon_ARJP11A-MASA-B-A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, J7 USB_C_Receptacle_PowerOnly_6P, SW1 NRST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

Commit message: Test Stage Added Pushbutton
Parts:
- added SW4: USER, Button_Switch_SMD:SW_Push_SPST_NO_Alps_SKRK, symbol Switch:SW_Push
Changed lines of the file:
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@@
+	)
+	(symbol
+		(lib_id "Switch:SW_Push")
+		(at 179.07 151.13 0)
+		(unit 1)
+		(exclude_from_sim no)
+		(in_bom yes)
+		(on_board yes)
+		(dnp no)
+		(fields_autoplaced yes)
+		(property "Reference" "SW4"
+			(at 179.07 143.51 0)
+			(effects
+				(font
+					(size 1.27 1.27)
+				)
+			)
+		)
+		(property "Value" "USER"
+			(at 179.07 146.05 0)
+			(effects
+				(font
+					(size 1.27 1.27)
+				)
+			)
+		)
+		(property "Footprint" "Button_Switch_SMD:SW_Push_SPST_NO_Alps_SKRK"
+			(at 179.07 146.05 0)
+			(effects
+				(font
+					(size 1.27 1.27)
+				)
+				(hide yes)
+			)
+		)
+		(property "Datasheet" "~"
+			(at 179.07 146.05 0)
+			(effects
+				(font
+					(size 1.27 1.27)
+				)
+				(hide yes)
+			)
+		)
+		(property "Description" "Push button switch, generic, two pins"
+			(at 179.07 151.13 0)
+			(effects
+				(font
+					(size 1.27 1.27)
+				)
+				(hide yes)
+			)
+		)
+		(pin "2"
+		)
+		(pin "1"
+		)
+		(instances
+			(project "20kN_dev"
+				(path "/b7d5eda3-9e79-4f11-b2ea-7bd3db80cdb6"
+					(reference "SW4")
+					(unit 1)
+				)
+			)
+		)
 	)
 	(symbol

Commit message: add a Wire
Connections:
- net at SW4.2: now also J5.6
Changed lines of the file:
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@@
+	(wire
+		(pts
+			(xy 184.15 151.13) (xy 227.33 151.13)
+		)
+		(stroke
+			(width 0)
+			(type default)
+		)
+	)
 	(wire
 		(pts
@@
 		)
 		(stroke
+			(width 0)
+			(type default)
+		)
+	)
+	(wire
+		(pts
+			(xy 227.33 151.13) (xy 227.33 132.08)
+		)
+		(stroke

Commit message: add GND Test
Connections:
- net GND: now also SW4.1
Changed lines of the file:
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@@
+	(wire
+		(pts
+			(xy 166.37 151.13) (xy 173.99 151.13)
+		)
+		(stroke
+			(width 0)
+			(type default)
+		)
+	)
 	(wire
 		(pts
@@
 		(pts
 			(xy 33.02 180.34) (xy 36.83 180.34)
+		)
+		(stroke
+			(width 0)
+			(type default)
+		)
+	)
+	(wire
+		(pts
+			(xy 166.37 158.75) (xy 166.37 151.13)
 		)
 		(stroke
@@
 					(unit 1)
 				)
+			)
+		)
+	)
+	(symbol
+		(lib_id "power:GND")
+		(at 166.37 158.75 0)
+		(unit 1)
+		(exclude_from_sim no)
+		(in_bom yes)
+		(on_board yes)
+		(dnp no)
+		(fields_autoplaced yes)
+		(property "Reference" "#PWR010"
+			(at 166.37 165.1 0)
+			(effects
+				(font
+					(size 1.27 1.27)
+				)
+				(hide yes)
+			)
+		)
+		(property "Value" "GND"
+			(at 166.37 163.83 0)
+			(effects
+				(font
+					(size 1.27 1.27)
+				)
+			)
+		)
+		(property "Footprint" ""
+			(at 166.37 158.75 0)
+			(effects
+				(font
+					(size 1.27 1.27)
+				)
+				(hide yes)
+			)
+		)
+		(property "Datasheet" ""
+			(at 166.37 158.75 0)
+			(effects
+				(font
+					(size 1.27 1.27)
+				)
+				(hide yes)
+			)
+		)
+		(property "Description" "Power symbol creates a global label with name \"GND\" , ground"
+			(at 166.37 158.75 0)
+			(effects
+				(font
+					(size 1.27 1.27)
+				)
+				(hide yes)
+			)
+		)
+		(pin "1"
+		)
+		(instances
+			(project ""
+				(path "/b7d5eda3-9e79-4f11-b2ea-7bd3db80cdb6"
+					(reference "#PWR010")
+					(unit 1)
+				)

Commit message: Test Branch Stepper Motor
Connections:
- net at IC2.13 (M0_/_APHASE): now also IC2.24 (VREFO)
Other:
- moved on the sheet: IC2
Changed lines of the file:
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@@
+	(wire
+		(pts
+			(xy 110.49 132.08) (xy 123.19 132.08)
+		)
+		(stroke
+			(width 0)
+			(type default)
+		)
+	)
 	(wire
 		(pts
@@
 	(wire
 		(pts
+			(xy 153.67 92.71) (xy 162.56 92.71)
+		)
+		(stroke
+			(width 0)
+			(type default)
+		)
+	)
+	(wire
+		(pts
 			(xy 167.64 128.27) (xy 170.18 128.27)
 		)
@@
 	(wire
 		(pts
+			(xy 148.59 104.14) (xy 153.67 104.14)
+		)
+		(stroke
+			(width 0)
+			(type default)
+		)
+	)
+	(wire
+		(pts
+			(xy 153.67 104.14) (xy 153.67 92.71)
+		)
+		(stroke
+			(width 0)
+			(type default)
+		)
+	)
+	(wire
+		(pts
 			(xy 34.29 167.64) (xy 34.29 165.1)
 		)
@@
 	(wire
 		(pts
+			(xy 162.56 76.2) (xy 148.59 76.2)
+		)
+		(stroke
+			(width 0)
+			(type default)
+		)
+	)
+	(wire
+		(pts
 			(xy 184.15 151.13) (xy 227.33 151.13)
 		)
@@
 	(wire
 		(pts
+			(xy 123.19 132.08) (xy 123.19 121.92)
+		)
+		(stroke
+			(width 0)
+			(type default)
+		)
+	)
+	(wire
+		(pts
 			(xy 86.36 160.02) (xy 86.36 157.48)
 		)
@@
 		(pts
 			(xy 34.29 170.18) (xy 36.83 170.18)
+		)
+		(stroke
+			(width 0)
+			(type default)
+		)
+	)
+	(wire
+		(pts
+			(xy 162.56 92.71) (xy 162.56 76.2)
 		)
 		(stroke
@@
 	(symbol
 		(lib_id "power:GND")
-		(at 124.46 111.76 0)
+		(at 110.49 132.08 0)
 		(unit 1)
 		(exclude_from_sim no)
@@
 		(fields_autoplaced yes)
 		(property "Reference" "#PWR02"
-			(at 124.46 118.11 0)
+			(at 110.49 138.43 0)
 			(effects
 				(font
@@
 		)
 		(property "Value" "GND"
-			(at 124.46 116.84 0)
+			(at 110.49 137.16 0)
 			(effects
 				(font
@@
 		)
 		(property "Footprint" ""
-			(at 124.46 111.76 0)
+			(at 110.49 132.08 0)
 			(effects
 				(font
@@
 		)
 		(property "Datasheet" ""
-			(at 124.46 111.76 0)
+			(at 110.49 132.08 0)
 			(effects
 				(font
@@
 		)
 		(property "Description" "Power symbol creates a global label with name \"GND\" , ground"
-			(at 124.46 111.76 0)
+			(at 110.49 132.08 0)
 			(effects
 				(font
@@
 	(symbol
 		(lib_id "Motor_Drive:DRV8834PWPR")
-		(at 99.06 66.04 0)
+		(at 97.79 76.2 0)
 		(unit 1)
 		(exclude_from_sim no)
@@
 		(fields_autoplaced yes)
 		(property "Reference" "IC2"
-			(at 124.46 58.42 0)
+			(at 123.19 68.58 0)
 			(effects
 				(font
@@
 		)
 		(property "Value" "DRV8834PWPR"
-			(at 124.46 60.96 0)
+			(at 123.19 71.12 0)
 			(effects
 				(font
@@
 		)
 		(property "Footprint" "Package_SO:HTSSOP-24-1EP_4.4x7.8mm_P0.65mm_EP3.2x5mm"
-			(at 146.05 160.96 0)
+			(at 144.78 171.12 0)
 			(effects
 				(font
@@
 		)
 		(property "Datasheet" "http://www.ti.com/lit/gpn/DRV8834"
-			(at 146.05 260.96 0)
+			(at 144.78 271.12 0)
 			(effects
 				(font
@@
 		)
 		(property "Description" "2.2A Low Voltage Stepper w/ 32-step Indexer or Dual Brushed DC Motor Driver (Indexer or PH/EN Ctrl)"
-			(at 119.38 54.356 0)
+			(at 118.11 64.516 0)
 			(effects
 				(font
@@
 		)
 		(property "Height" "1.2"
-			(at 146.05 460.96 0)
+			(at 144.78 471.12 0)
 			(effects
 				(font
@@
 		)
 		(property "Mouser Part Number" "595-DRV8834PWPR"
-			(at 146.05 560.96 0)
+			(at 144.78 571.12 0)
 			(effects
 				(font
@@
 		)
 		(property "Mouser Price/Stock" "https://www.mouser.co.uk/ProductDetail/Texas-Instruments/DRV8834PWPR?qs=UFc95S4Z4CYJbHHHrd3TVA%3D%3D"
-			(at 146.05 660.96 0)
+			(at 144.78 671.12 0)
 			(effects
 				(font
@@
 		)
 		(property "Manufacturer_Name" "Texas Instruments"
-			(at 146.05 760.96 0)
+			(at 144.78 771.12 0)
 			(effects
 				(font
@@
 		)
 		(property "Manufacturer_Part_Number" "DRV8834PWPR"
-			(at 146.05 860.96 0)
-			(effects
-				(font
+			(at 144.78 871.12 0)
+			(effects
+				(font

Commit message: change Stepper Test
Connections:
- net at IC2.13 (M0_/_APHASE): no longer IC2.24 (VREFO)
Changed lines of the file:
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@@
-	(wire
-		(pts
-			(xy 153.67 92.71) (xy 162.56 92.71)
-		)
-		(stroke
-			(width 0)
-			(type default)
-		)
-	)
 	(wire
 		(pts
@@
 	(wire
 		(pts
-			(xy 148.59 104.14) (xy 153.67 104.14)
-		)
-		(stroke
-			(width 0)
-			(type default)
-		)
-	)
-	(wire
-		(pts
-			(xy 153.67 104.14) (xy 153.67 92.71)
-		)
-		(stroke
-			(width 0)
-			(type default)
-		)
-	)
-	(wire
-		(pts
 			(xy 34.29 167.64) (xy 34.29 165.1)
 		)
@@
 		(pts
 			(xy 34.29 172.72) (xy 34.29 177.8)
-		)
-		(stroke
-			(width 0)
-			(type default)
-		)
-	)
-	(wire
-		(pts
-			(xy 162.56 76.2) (xy 148.59 76.2)
 		)
 		(stroke
@@
 		)
 		(stroke
-			(width 0)
-			(type default)
-		)
-	)
-	(wire
-		(pts
-			(xy 162.56 92.71) (xy 162.56 76.2)
-		)
-		(stroke
